File: src/ch340.sch (KiCad schematic (older format))
At the start: 17 parts, among them J1 USB_A, J2 Conn_01x04_Male, U1 CH340C, U2 662K

Commit message: 1. set track width of GND, VCC 0.5mm 2. add vias to GND 3. change footprint, 0403 to 0603 handsoldering
Parts:
- C1, C2: footprint Capacitor_SMD:C_0603_1608Metric -> Capacitor_SMD:C_0603_1608Metric_Pad1.08x0.95mm_HandSolder
- C3, C4: footprint Capacitor_SMD:C_0402_1005Metric -> Capacitor_SMD:C_0603_1608Metric_Pad1.08x0.95mm_HandSolder
- D1, D2, D3: footprint LED_SMD:LED_0603_1608Metric -> LED_SMD:LED_0603_1608Metric_Pad1.05x0.95mm_HandSolder
- R1, R2: footprint Resistor_SMD:R_0402_1005Metric -> Resistor_SMD:R_0603_1608Metric_Pad0.98x0.95mm_HandSolder
- R3, R4, R5: footprint Resistor_SMD:R_0603_1608Metric -> Resistor_SMD:R_0603_1608Metric_Pad0.98x0.95mm_HandSolder
- U2: footprint Package_TO_SOT_SMD:SOT-23 -> Package_TO_SOT_SMD:SOT-23_Handsoldering
Changed lines of the file:
@@
 F 0 "C1" H 4615 4346 50  0000 L CNN
 F 1 "0.1uF" H 4615 4255 50  0000 L CNN
-F 2 "Capacitor_SMD:C_0603_1608Metric" H 4538 4150 50  0001 C CNN
+F 2 "Capacitor_SMD:C_0603_1608Metric_Pad1.08x0.95mm_HandSolder" H 4538 4150 50  0001 C CNN
 F 3 "~" H 4500 4300 50  0001 C CNN
 	1    4500 4300
@@
 F 0 "C2" H 4915 4346 50  0000 L CNN
 F 1 "0.1uF" H 4915 4255 50  0000 L CNN
-F 2 "Capacitor_SMD:C_0603_1608Metric" H 4838 4150 50  0001 C CNN
+F 2 "Capacitor_SMD:C_0603_1608Metric_Pad1.08x0.95mm_HandSolder" H 4838 4150 50  0001 C CNN
 F 3 "~" H 4800 4300 50  0001 C CNN
 	1    4800 4300
@@
 F 0 "R1" V 6250 4400 50  0000 C CNN
 F 1 "200R" V 6250 4650 50  0000 C CNN
-F 2 "Resistor_SMD:R_0402_1005Metric" V 6280 4500 50  0001 C CNN
+F 2 "Resistor_SMD:R_0603_1608Metric_Pad0.98x0.95mm_HandSolder" V 6280 4500 50  0001 C CNN
 F 3 "~" H 6350 4500 50  0001 C CNN
 	1    6350 4500
@@
 F 0 "R2" V 6450 4500 50  0000 C CNN
 F 1 "200R" V 6450 4750 50  0000 C CNN
-F 2 "Resistor_SMD:R_0402_1005Metric" V 6280 4600 50  0001 C CNN
+F 2 "Resistor_SMD:R_0603_1608Metric_Pad0.98x0.95mm_HandSolder" V 6280 4600 50  0001 C CNN
 F 3 "~" H 6350 4600 50  0001 C CNN
 	1    6350 4600
@@
 F 0 "U2" H 4450 2865 50  0000 C CNN
 F 1 "662K" H 4450 2774 50  0000 C CNN
-F 2 "Package_TO_SOT_SMD:SOT-23" H 4450 2200 50  0001 C CNN
+F 2 "Package_TO_SOT_SMD:SOT-23_Handsoldering" H 4450 2200 50  0001 C CNN
 F 3 "" H 4300 2700 50  0001 C CNN
 	1    4450 2500
@@
 F 0 "C3" H 3965 2646 50  0000 L CNN
 F 1 "1uF" H 3965 2555 50  0000 L CNN
-F 2 "Capacitor_SMD:C_0402_1005Metric" H 3888 2450 50  0001 C CNN
+F 2 "Capacitor_SMD:C_0603_1608Metric_Pad1.08x0.95mm_HandSolder" H 3888 2450 50  0001 C CNN
 F 3 "~" H 3850 2600 50  0001 C CNN
 	1    3850 2600
@@
 F 0 "C4" H 5265 2646 50  0000 L CNN
 F 1 "1uF" H 5265 2555 50  0000 L CNN
-F 2 "Capacitor_SMD:C_0402_1005Metric" H 5188 2450 50  0001 C CNN
+F 2 "Capacitor_SMD:C_0603_1608Metric_Pad1.08x0.95mm_HandSolder" H 5188 2450 50  0001 C CNN
 F 3 "~" H 5150 2600 50  0001 C CNN
 	1    5150 2600
@@
 F 0 "R3" H 6230 2304 50  0000 R CNN
 F 1 "1K" H 6230 2395 50  0000 R CNN
-F 2 "Resistor_SMD:R_0603_1608Metric" V 6230 2350 50  0001 C CNN
+F 2 "Resistor_SMD:R_0603_1608Metric_Pad0.98x0.95mm_HandSolder" V 6230 2350 50  0001 C CNN
 F 3 "~" H 6300 2350 50  0001 C CNN
 	1    6300 2350
@@
 F 0 "D1" V 6339 2582 50  0000 R CNN
 F 1 "LED RED" V 6248 2582 50  0000 R CNN
-F 2 "LED_SMD:LED_0603_1608Metric" H 6300 2700 50  0001 C CNN
+F 2 "LED_SMD:LED_0603_1608Metric_Pad1.05x0.95mm_HandSolder" H 6300 2700 50  0001 C CNN
 F 3 "~" H 6300 2700 50  0001 C CNN
 	1    6300 2700
@@
 F 0 "R4" H 6830 2304 50  0000 R CNN
 F 1 "1K" H 6830 2395 50  0000 R CNN
-F 2 "Resistor_SMD:R_0603_1608Metric" V 6830 2350 50  0001 C CNN
+F 2 "Resistor_SMD:R_0603_1608Metric_Pad0.98x0.95mm_HandSolder" V 6830 2350 50  0001 C CNN
 F 3 "~" H 6900 2350 50  0001 C CNN
 	1    6900 2350
@@
 F 0 "D2" V 6939 2582 50  0000 R CNN
 F 1 "LED GREEN" V 6848 2582 50  0000 R CNN
-F 2 "LED_SMD:LED_0603_1608Metric" H 6900 2700 50  0001 C CNN
+F 2 "LED_SMD:LED_0603_1608Metric_Pad1.05x0.95mm_HandSolder" H 6900 2700 50  0001 C CNN
 F 3 "~" H 6900 2700 50  0001 C CNN
 	1    6900 2700
@@
 F 0 "R5" H 7430 2304 50  0000 R CNN
 F 1 "1K" H 7430 2395 50  0000 R CNN
-F 2 "Resistor_SMD:R_0603_1608Metric" V 7430 2350 50  0001 C CNN
+F 2 "Resistor_SMD:R_0603_1608Metric_Pad0.98x0.95mm_HandSolder" V 7430 2350 50  0001 C CNN
 F 3 "~" H 7500 2350 50  0001 C CNN
 	1    7500 2350
@@
 F 0 "D3" V 7539 2582 50  0000 R CNN
 F 1 "LED GREEN" V 7448 2582 50  0000 R CNN
-F 2 "LED_SMD:LED_0603_1608Metric" H 7500 2700 50  0001 C CNN
+F 2 "LED_SMD:LED_0603_1608Metric_Pad1.05x0.95mm_HandSolder" H 7500 2700 50  0001 C CNN
 F 3 "~" H 7500 2700 50  0001 C CNN
 	1    7500 2700
